Commit message: Add shitty project zip

File: boro.urdf (robot description, URDF)
Before this commit: robot boro, 4 links, 3 joints
Links:
- added link bow_contact_frame
- link link1: mass None -> 0.1703
- link link2: mass None -> 0.3405; geometry visual cylinder length=0.8 radius=0.01
- link link3: mass 0.2 -> 0.5108; geometry visual cylinder length=0.6 radius=0.01
Joints:
- added joint bow_contact_frame_joint: type fixed, parent link3, child bow_contact_frame, origin xyz=0.05 0 0 rpy=3.141592653589793 -1.57079632679 0
- joint joint_h: limit (none) -> lower=-0.1 upper=0.1 effort=0 velocity=0; origin xyz=0 0 0.1 rpy=0 0 0 -> xyz=0 -0.1 0 rpy=1.57079632679 0 0
- joint joint_l: axis 1 0 0 -> 0 0 1; limit lower=0 upper=0.3 -> lower=-0.4 upper=0.4 effort=0 velocity=0; origin xyz=0 0 0 rpy=0 0 0 -> xyz=0.4 0 0 rpy=0 1.57079632679 0
- joint joint_phi: axis 0 1 0 -> 0 0 1; limit lower=-0.79 upper=0.79 -> lower=-0.79 upper=0.79 effort=0 velocity=0; origin xyz=0 0 0 -> xyz=0 0 0.3 rpy=-1.57079632679 0 0
